File: main.kicad_pcb (KiCad board)
At the start: 2 copper layers, 21.3 x 40.6 mm, 3 parts, among them J1 USB_A, J2 USB_A, J3 OrangePiCon

Commit message: outline update
Parts:
- moved J2 1.27 mm to (247.4, 156.2)
Other:
- outline, holes or cut-outs redrawn
